File: kicad/nRF24.kicad_pcb (KiCad board)
At the start: 2 copper layers, 20 parts, among them J1 Conn_Coaxial, J2 Conn_01x08, U1 nRF24L01P, X2 16MHz

Commit message: add rfx2401c
Parts:
- removed X2: 16MHz, Crystal:Crystal_HC52-U_Vertical
- added C12: 10uF, Capacitor_SMD:C_0603_1608Metric, F.Cu at (73.0, 35.0)
- added C13: 100nF, Capacitor_SMD:C_0603_1608Metric, F.Cu at (75.0, 35.0)
- added C14: 10uF, Capacitor_SMD:C_0603_1608Metric, F.Cu at (65.0, 35.0)
- added C15: 100nF, Capacitor_SMD:C_0603_1608Metric, F.Cu at (67.0, 35.0)
- added C16: 1uF, Capacitor_SMD:C_0603_1608Metric, F.Cu at (57.6, 49.2)
- added C17: 10uF, Capacitor_SMD:C_0603_1608Metric, F.Cu at (55.6, 49.2)
- added C18: 0.3pF, Capacitor_SMD:C_0603_1608Metric, F.Cu at (52.7, 44.2)
- added C19: 1.5pF, Capacitor_SMD:C_0603_1608Metric, F.Cu at (51.1, 44.2)
- added C20: 1.5pF, Capacitor_SMD:C_0603_1608Metric, F.Cu at (46.3, 44.2)
- added C21: 1.5pF, Capacitor_SMD:C_0603_1608Metric, F.Cu at (44.7, 44.2)
- added C22: 1.5pF, Capacitor_SMD:C_0603_1608Metric, F.Cu at (39.9, 44.2)
- added H1: MountingHole, MountingHole:MountingHole_3.2mm_M3, F.Cu at (35.0, 35.0)
- added H2: MountingHole, MountingHole:MountingHole_3.2mm_M3, F.Cu at (35.0, 55.0)
- added L4: 2.4nH, Inductor_SMD:L_0603_1608Metric, F.Cu at (48.7, 45.2)
- added L5: 2.4nH, Inductor_SMD:L_0603_1608Metric, F.Cu at (42.3, 45.2)
- added R3: 10k, Resistor_SMD:R_0603_1608Metric, F.Cu at (54.0, 41.0)
- added R4: 1k, Resistor_SMD:R_0603_1608Metric, F.Cu at (55.6, 41.0)
- added R5: 1k, Resistor_SMD:R_0603_1608Metric, F.Cu at (57.2, 41.0)
- added U2: TLV75733PDBV, Package_TO_SOT_SMD:SOT-23-5, F.Cu at (70.0, 35.0)
- added U3: RFX2401C, RFX2401C:QFN-16_L3.0-W3.0-P0.50-BL-EP1.7, F.Cu at (55.5, 45.2)
- added X1: 16MHz, Crystal:Crystal_HC52-U_Vertical, F.Cu at (54.1, 34.0)
- C10: value 15pF -> 22pF
- C11: value 1.5pF -> 22pF
- C6: value 22pF -> 2.2nF
- C7: value 2.2nF -> 4.7pF
- C8: value 4.7pF -> 15pF
- C9: value 22pF -> 1.5pF
- J1: value Conn_Coaxial -> Conn_01x08; footprint Connector_Coaxial:SMA_Amphenol_901-143_Horizontal -> Connector_PinHeader_2.54mm:PinHeader_1x08_P2.54mm_Vertical
- J2: value Conn_01x08 -> Conn_Coaxial; footprint Connector_PinHeader_2.54mm:PinHeader_1x08_P2.54mm_Vertical -> Connector_Coaxial:SMA_Amphenol_901-143_Horizontal
- L1: value 12nH -> 2.3nH
- L2: value 2.3nH -> 12nH
- moved J2 104.8 mm to (34.5, 45.0), turned to 90 degrees
- moved C10 70.6 mm to (49.8, 34.0), turned to 180 degrees
- moved R2 69.2 mm to (56.0, 31.0)
- moved C9 60.4 mm to (58.5, 44.9), turned to -90 degrees
- moved C11 59.2 mm to (62.2, 34.0)
- moved L3 59.0 mm to (64.0, 45.7), turned to 180 degrees
- moved C8 58.1 mm to (60.9, 45.7), turned to 180 degrees
- moved L2 56.8 mm to (66.3, 44.9), turned to -90 degrees
- moved R1 55.1 mm to (68.0, 50.2), turned to -90 degrees
- moved C7 54.2 mm to (64.7, 41.8), turned to 90 degrees
- moved L1 53.9 mm to (66.3, 41.8), turned to -90 degrees
- moved C6 53.1 mm to (63.1, 41.8), turned to 90 degrees
- moved J1 51.8 mm to (78.0, 53.9), turned to 180 degrees
- moved C3 48.8 mm to (66.3, 50.2), turned to -90 degrees
- moved U1 48.1 mm to (70.0, 45.2), turned to 180 degrees
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Connections:
- C1 pad 1: /Connector/VCC -> +3.3V
- C10 pad 1: Net-(C10-Pad1) -> XTAL_N
- C10 pad 2: Net-(J1-In) -> GND
- C11 pad 1: GND -> XTAL_P
- C11 pad 2: Net-(J1-In) -> GND
- C2 pad 1: /Connector/VCC -> +3.3V
- C3 pad 1: /Connector/VCC -> +3.3V
- C5 pad 1: /Connector/VCC -> +3.3V
- C6 pad 1: Net-(U1-XC2) -> GND
- C6 pad 2: GND -> /PA_LNA/VDD_PA
- C7 pad 2: Net-(U1-VDD_PA) -> /PA_LNA/VDD_PA
- C8 pad 1: GND -> Net-(C8-Pad1)
- C8 pad 2: Net-(U1-VDD_PA) -> /PA_LNA/RF
- C9 pad 1: Net-(U1-XC1) -> GND
- C9 pad 2: GND -> /PA_LNA/RF
- J1 pad 1: Net-(J1-In) -> GND
- J1 pad 2: GND -> VIN
- J2 pad 1: GND -> /PA_LNA/ANT
- J2 pad 2: /Connector/VCC -> GND
- L1 pad 1: Net-(U1-ANT1) -> /PA_LNA/VDD_PA
- L1 pad 2: Net-(U1-ANT2) -> Net-(U1-ANT1)
- L2 pad 1: Net-(U1-VDD_PA) -> Net-(U1-ANT1)
- L2 pad 2: Net-(U1-ANT1) -> Net-(U1-ANT2)
- L3 pad 2: Net-(C10-Pad1) -> Net-(C8-Pad1)
- R2 pad 1: Net-(U1-XC2) -> XTAL_N
- R2 pad 2: Net-(U1-XC1) -> XTAL_P
- U1 pad 10: Net-(U1-XC1) -> XTAL_N
- U1 pad 11: Net-(U1-VDD_PA) -> /PA_LNA/VDD_PA
- U1 pad 15: /Connector/VCC -> +3.3V
- U1 pad 18: /Connector/VCC -> +3.3V
- U1 pad 7: /Connector/VCC -> +3.3V
- U1 pad 9: Net-(U1-XC2) -> XTAL_P
Routing:
- net +3.3V: track 0.00 -> 52.7 mm, vias 0 -> 2
- net /Connector/CE: track 0.00 -> 37.5 mm, vias 0 -> 1
- net VIN: track 0.00 -> 27.3 mm, vias 0 -> 1
- net XTAL_N: track 0.00 -> 26.1 mm
- net XTAL_P: track 0.00 -> 24.8 mm
- net /PA_LNA/VDD_PA: track 0.00 -> 13.4 mm
- net /Connector/IRQ: track 0.00 -> 10.1 mm
- net /Connector/MISO: track 0.00 -> 8.37 mm
- net /Connector/MOSI: track 0.00 -> 7.53 mm
- net /PA_LNA/ANT: track 0.00 -> 7.11 mm
- net /Connector/SCK: track 0.00 -> 6.68 mm
- net /Connector/CSN: track 0.00 -> 6.29 mm
- net Net-(FL1-IN): track 0.00 -> 5.01 mm
- net Net-(FL1-OUT): track 0.00 -> 4.72 mm
- net /PA_LNA/RF: track 0.00 -> 3.86 mm
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- added copper zone on B.Cu, net GND
- added copper zone on F.Cu, net GND
Other:
- board outline added: 50 x 30 mm
- board text added: "CE"
- board text added: "GND"
- board text added: "IRQ"
- board text added: "MISO"
- board text added: "MOSI"
- board text added: "SCK"
- board text added: "VIN"
- board text added: "~{CS}"
