File: kicad/nRF24.kicad_pcb (KiCad board)
At the start: 2 copper layers, 50 x 30 mm, 40 parts, among them J1 Conn_01x08, J2 Conn_Coaxial, U1 nRF24L01P, U2 TLV75733PDBV, U3 RFX2401C, X1 16MHz

Commit message: add graph
Routing:
- net +3.3V: track 52.7 -> 31.0 mm, vias 2 -> 4
- added copper zone on In2.Cu, net +3.3V
- added copper zone on In1.Cu, net GND
Other:
- copper layers 2 -> 4
Changed lines of the file:
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@@
 	(generator_version "10.0")
 	(general
-		(thickness 1.6)
+		(thickness 1.6062)
 		(legacy_teardrops no)
 	)
@@
 	(layers
 		(0 "F.Cu" signal)
+		(4 "In1.Cu" signal)
+		(6 "In2.Cu" signal)
 		(2 "B.Cu" signal)
 		(9 "F.Adhes" user "F.Adhesive")
@@
 			)
 			(layer "dielectric 1"
+				(type "prepreg")
+				(thickness 0.2104)
+				(material "FR4")
+				(epsilon_r 4.5)
+				(loss_tangent 0.02)
+			)
+			(layer "In1.Cu"
+				(type "copper")
+				(thickness 0.0152)
+			)
+			(layer "dielectric 2"
 				(type "core")
-				(thickness 1.51)
+				(thickness 1.065)
+				(material "FR4")
+				(epsilon_r 4.5)
+				(loss_tangent 0.02)
+			)
+			(layer "In2.Cu"
+				(type "copper")
+				(thickness 0.0152)
+			)
+			(layer "dielectric 3"
+				(type "prepreg")
+				(thickness 0.2104)
 				(material "FR4")
 				(epsilon_r 4.5)
@@
 			(remove_unused_layers yes)
 			(keep_end_layers yes)
-			(zone_layer_connections)
+			(zone_layer_connections "In1.Cu")
 			(net "GND")
 			(pinfunction "Ext_2")
@@
 			(remove_unused_layers yes)
 			(keep_end_layers yes)
-			(zone_layer_connections)
+			(zone_layer_connections "In1.Cu")
 			(net "GND")
 			(pinfunction "Ext_2")
@@
 			(remove_unused_layers yes)
 			(keep_end_layers yes)
-			(zone_layer_connections)
+			(zone_layer_connections "In1.Cu")
 			(net "GND")
 			(pinfunction "Ext_2")
@@
 			(remove_unused_layers yes)
 			(keep_end_layers yes)
-			(zone_layer_connections)
+			(zone_layer_connections "In1.Cu")
 			(net "GND")
 			(pinfunction "Ext_2")
@@
 	)
 	(segment
-		(start 65.5 48.6144)
-		(end 58.803 48.6144)
+		(start 70.55 41)
+		(end 69 41)
 		(width 0.5)
 		(layer "F.Cu")
@@
 	)
 	(segment
+		(start 58.5 48.45)
+		(end 58.9 48.85)
+		(width 0.5)
+		(layer "F.Cu")
+		(net "+3.3V")
+	)
+	(segment
 		(start 67.05 50.2)
 		(end 68.95 50.2)
@@
 	(segment
 		(start 65 35.775)
+		(end 64.225 35.775)
+		(width 0.5)
+		(layer "F.Cu")
+		(net "+3.3V")
+	)
+	(segment
+		(start 65 35.775)
 		(end 67 35.775)
 		(width 0.5)
@@
 	)
 	(segment
+		(start 64.225 35.775)
+		(end 64 36)
+		(width 0.5)
+		(layer "F.Cu")
+		(net "+3.3V")
+	)
+	(segment
+		(start 57.65 48.45)
+		(end 58.5 48.45)
+		(width 0.5)
+		(layer "F.Cu")
+		(net "+3.3V")
+	)
+	(segment
 		(start 67 35.775)
 		(end 68.6875 35.775)
@@
 	)
 	(segment
-		(start 65 35.775)
-		(end 70 40.775)
-		(width 0.5)
-		(layer "F.Cu")
-		(net "+3.3V")
-	)
-	(segment
 		(start 70 49.15)
 		(end 69.7 49.45)
@@
 	)
 	(segment
-		(start 68.3125 39.0875)
-		(end 68.3283 39.1033)
-		(width 0.2)
+		(start 70 41)
+		(end 70.55 41)
+		(width 0.5)
 		(layer "F.Cu")
 		(net "+3.3V")
@@
 	)
 	(segment
-		(start 70 41)
+		(start 70.55 41)
 		(end 72 41)
 		(width 0.5)
@@
 	)
 	(segment
-		(start 58.6386 48.45)
-		(end 57.65 48.45)
-		(width 0.5)
-		(layer "F.Cu")
-		(net "+3.3V")
-	)
-	(segment
 		(start 66.3 49.45)
 		(end 66.3 47.4)
@@
 		(net "+3.3V")
 	)
-	(segment
-		(start 58.803 48.6144)
-		(end 58.6386 48.45)
-		(width 0.5)
-		(layer "F.Cu")
-		(net "+3.3V")
-	)
 	(via
-		(at 68.3125 39.0875)
+		(at 69 41)
 		(size 0.6)
 		(drill 0.3)
@@
 	)
 	(via
-		(at 65.5 48.6144)
+		(at 64 36)
 		(size 0.6)
 		(drill 0.3)
@@
 		(net "+3.3V")
 	)
-	(segment
-		(start 65.5 41.9174)
-		(end 65.5 48.6144)
-		(width 0.5)
-		(layer "B.Cu")
-		(net "+3.3V")
-	)
-	(segment
-		(start 68.3125 39.0875)
-		(end 67.6 39.8)
-		(width 0.5)
-		(layer "B.Cu")
-		(net "+3.3V")
-	)
-	(segment
-		(start 67.6 39.8174)
-		(end 65.5 41.9174)
-		(width 0.5)
-		(layer "B.Cu")
+	(via
+		(at 58.9 48.85)
+		(size 0.6)
+		(drill 0.3)
+		(layers "F.Cu" "B.Cu")
 		(net "+3.3V")
 	)
-	(segment
-		(start 67.6 39.8)
-		(end 67.6 39.8174)
-		(width 0.5)
-		(layer "B.Cu")
+	(via
+		(at 65.5 48.6144)
+		(size 0.6)
+		(drill 0.3)
+		(layers "F.Cu" "B.Cu")
 		(net "+3.3V")
 	)
@@
 	(zone
 		(net "GND")
-		(layers "F.Cu" "B.Cu")
+		(layers "F.Cu" "B.Cu" "In1.Cu")
+		(hatch edge 0.5)
+		(connect_pads yes
+			(clearance 0.1)
+		)
+		(min_thickness 0.25)
+		(fill yes
+			(thermal_gap 0.5)
+			(thermal_bridge_width 0.5)
+			(island_removal_mode 0)
+		)
+		(polygon
+			(pts
+				(xy 30 30) (xy 80 30) (xy 80 60) (xy 30 60)
+			)
+		)
+	)
+	(zone
+		(net "+3.3V")
+		(layer "In2.Cu")
 		(hatch edge 0.5)
+		(priority 1)
 		(connect_pads yes
 			(clearance 0.1)

Commit message: journal images and reamde
Parts:
- L1, L3: footprint Inductor_SMD:L_0603_1608Metric -> Inductor_SMD:L_0402_1005Metric
Changed lines of the file:
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@@
 		)
 	)
-	(footprint "Inductor_SMD:L_0603_1608Metric"
+	(footprint "Inductor_SMD:L_0402_1005Metric"
 		(layer "F.Cu")
 		(at 66.3 41.825 -90)
-		(descr "Inductor SMD 0603 (1608 Metric), square (rectangular) end terminal, IPC-7351 nominal, (Body size source: http://www.tortai-tech.com/upload/download/2011102023233369053.pdf)")
+		(descr "Inductor SMD 0402 (1005 Metric), square (rectangular) end terminal, IPC-7351 nominal, (Body size source: http://www.tortai-tech.com/upload/download/2011102023233369053.pdf)")
 		(tags "inductor")
 		(property "Reference" "L1"
-			(at 0 -1.43 90)
+			(at 0 -1.17 270)
 			(layer "F.SilkS")
 			(effects
@@
 		)
 		(property "Value" "2.3nH"
-			(at 0 1.43 90)
+			(at 0 1.17 270)
 			(layer "F.Fab")
 			(effects
@@
 		)
 		(property "Datasheet" ""
-			(at 0 0 90)
+			(at 0 0 270)
 			(layer "F.Fab")
 			(hide yes)
@@
 		)
 		(property "Description" "Inductor, small symbol"
-			(at 0 0 90)
+			(at 0 0 270)
 			(layer "F.Fab")
 			(hide yes)
@@
 		)
 		(property "KiLib_Generator" "SMD_2terminal_chip_molded"
-			(at 0 0 90)
+			(at 0 0 270)
 			(layer "F.SilkS")
 			(hide yes)
@@
 		(attr smd)
 		(duplicate_pad_numbers_are_jumpers no)
-		(fp_line
-			(start -0.16278 0.51)
-			(end 0.16278 0.51)
-			(stroke
-				(width 0.12)
-				(type solid)
-			)
-			(layer "F.SilkS")
-		)
-		(fp_line
-			(start -0.16278 -0.51)
-			(end 0.16278 -0.51)
-			(stroke
-				(width 0.12)
-				(type solid)
-			)
-			(layer "F.SilkS")
-		)
-		(fp_poly
-			(pts
-				(xy -1.48 -0.73) (xy 1.48 -0.73) (xy 1.48 0.73) (xy -1.48 0.73)
-			)
+		(fp_rect
+			(start -0.93 -0.47)
+			(end 0.93 0.47)
 			(stroke
 				(width 0.05)
@@
 			(layer "F.CrtYd")
 		)
-		(fp_poly
-			(pts
-				(xy -0.8 -0.4) (xy 0.8 -0.4) (xy 0.8 0.4) (xy -0.8 0.4)
-			)
+		(fp_rect
+			(start -0.5 -0.25)
+			(end 0.5 0.25)
 			(stroke
 				(width 0.1)
@@
 		)
 		(fp_text user "${REFERENCE}"
-			(at 0 0 90)
+			(at 0 0 270)
 			(layer "F.Fab")
 			(effects
 				(font
-					(size 0.4 0.4)
-					(thickness 0.06)
+					(size 0.25 0.25)
+					(thickness 0.04)
 				)
 			)
 		)
 		(pad "1" smd roundrect
-			(at -0.787501 0 270)
-			(size 0.875 0.95)
+			(at -0.485 0 270)
+			(size 0.59 0.64)
 			(layers "F.Cu" "F.Mask" "F.Paste")
 			(roundrect_rratio 0.25)
@@
 		)
 		(pad "2" smd roundrect
-			(at 0.787501 0 270)
-			(size 0.875 0.95)
+			(at 0.485 0 270)
+			(size 0.59 0.64)
 			(layers "F.Cu" "F.Mask" "F.Paste")
 			(roundrect_rratio 0.25)
@@
 		)
 		(embedded_fonts no)
-		(model "${KICAD10_3DMODEL_DIR}/Inductor_SMD.3dshapes/L_0603_1608Metric.step"
+		(model "${KICAD10_3DMODEL_DIR}/Inductor_SMD.3dshapes/L_0402_1005Metric.step"
 			(offset
 				(xyz 0 0 0)
@@
 		)
 	)
-	(footprint "Inductor_SMD:L_0603_1608Metric"
+	(footprint "Inductor_SMD:L_0402_1005Metric"
 		(layer "F.Cu")
 		(at 64 45.725 180)
-		(descr "Inductor SMD 0603 (1608 Metric), square (rectangular) end terminal, IPC-7351 nominal, (Body size source: http://www.tortai-tech.com/upload/download/2011102023233369053.pdf)")
+		(descr "Inductor SMD 0402 (1005 Metric), square (rectangular) end terminal, IPC-7351 nominal, (Body size source: http://www.tortai-tech.com/upload/download/2011102023233369053.pdf)")
 		(tags "inductor")
 		(property "Reference" "L3"
-			(at 0 -1.43 0)
+			(at 0 -1.17 180)
 			(layer "F.SilkS")
 			(effects
@@
 		)
 		(property "Value" "7.9nH"
-			(at 0 1.43 0)
+			(at 0 1.17 180)
 			(layer "F.Fab")
 			(effects
@@
 		)
 		(property "Datasheet" ""
-			(at 0 0 0)
+			(at 0 0 180)
 			(layer "F.Fab")
 			(hide yes)
@@
 		)
 		(property "Description" "Inductor, small symbol"
-			(at 0 0 0)
+			(at 0 0 180)
 			(layer "F.Fab")
 			(hide yes)
@@
 		)
 		(property "KiLib_Generator" "SMD_2terminal_chip_molded"
-			(at 0 0 0)
+			(at 0 0 180)
 			(layer "F.SilkS")
 			(hide yes)
@@
 		(attr smd)
 		(duplicate_pad_numbers_are_jumpers no)
-		(fp_line
-			(start -0.16278 0.51)
-			(end 0.16278 0.51)
-			(stroke
-				(width 0.12)
-				(type solid)
-			)
-			(layer "F.SilkS")
-		)
-		(fp_line
-			(start -0.16278 -0.51)
-			(end 0.16278 -0.51)
-			(stroke
-				(width 0.12)
-				(type solid)
-			)
-			(layer "F.SilkS")
-		)
-		(fp_poly
-			(pts
-				(xy -1.48 -0.73) (xy 1.48 -0.73) (xy 1.48 0.73) (xy -1.48 0.73)
-			)
+		(fp_rect
+			(start -0.93 -0.47)
+			(end 0.93 0.47)
 			(stroke
 				(width 0.05)
@@
 			(layer "F.CrtYd")
 		)
-		(fp_poly
-			(pts
-				(xy -0.8 -0.4) (xy 0.8 -0.4) (xy 0.8 0.4) (xy -0.8 0.4)
-			)
+		(fp_rect
+			(start -0.5 -0.25)
+			(end 0.5 0.25)
 			(stroke
 				(width 0.1)
@@
 		)
 		(fp_text user "${REFERENCE}"
-			(at 0 0 0)
+			(at 0 0 180)
 			(layer "F.Fab")
 			(effects
 				(font
-					(size 0.4 0.4)
-					(thickness 0.06)
+					(size 0.25 0.25)
+					(thickness 0.04)
 				)
 			)
 		)
 		(pad "1" smd roundrect
-			(at -0.787501 0 180)
-			(size 0.875 0.95)
+			(at -0.485 0 180)
+			(size 0.59 0.64)
 			(layers "F.Cu" "F.Mask" "F.Paste")
 			(roundrect_rratio 0.25)
@@
 		)
 		(pad "2" smd roundrect
-			(at 0.787501 0 180)
-			(size 0.875 0.95)
+			(at 0.485 0 180)
+			(size 0.59 0.64)
 			(layers "F.Cu" "F.Mask" "F.Paste")
 			(roundrect_rratio 0.25)
@@
 		)
 		(embedded_fonts no)
-		(model "${KICAD10_3DMODEL_DIR}/Inductor_SMD.3dshapes/L_0603_1608Metric.step"
+		(model "${KICAD10_3DMODEL_DIR}/Inductor_SMD.3dshapes/L_0402_1005Metric.step"
 			(offset
 				(xyz 0 0 0)
