File: kicad/connector.kicad_sch (KiCad schematic)
At the start: 1 part, among them J2 Conn_01x08

Commit message: journal and image
Parts:
- added C10, C12: 10uF, symbol Device:C_Small
- added C11, C13: 100nF, symbol Device:C_Small
- added U2: TLV75733PDBV, Package_TO_SOT_SMD:SOT-23-5, symbol Regulator_Linear:TLV75733PDBV
- renumbered J2 to J1
Connections:
- net GND: now also C10.2, C11.2, C12.2, C13.2, U2.2 (GND)
- net VCC: now also C12.1, C13.1, U2.5 (OUT); no longer J1.2 (Pin_2)
- new net VIN: C10.1, C11.1, J1.2 (Pin_2), U2.1 (IN), U2.3 (EN)

Commit message: add rfx2401c
Parts:
- C12: renamed from C10; footprint (none) -> Capacitor_SMD:C_0603_1608Metric
- C13: renamed from C11; footprint (none) -> Capacitor_SMD:C_0603_1608Metric
- C14: renamed from C12; footprint (none) -> Capacitor_SMD:C_0603_1608Metric
- C15: renamed from C13; footprint (none) -> Capacitor_SMD:C_0603_1608Metric
Connections:
- net VCC renamed +3.3V
