File: kicad/rfconn.kicad_sch (KiCad schematic)
At the start: 4 parts, among them J2 Conn_Coaxial

Commit message: add rfx2401c
Parts:
- removed C14: 15pF, Capacitor_SMD:C_0603_1608Metric, symbol Device:C_Small
- removed C15: 1.5pF, Capacitor_SMD:C_0603_1608Metric, symbol Device:C_Small
- removed L3: 7.9nH, Inductor_SMD:L_0603_1608Metric, symbol Device:L_Small
Connections:
- net ANT: now also J2.1 (In)
